File: eagle/lib/thermoscheme.sch (EAGLE design)
At the start: 14 parts, among them U1 MLX90640ESF-BAB-000-TU

Commit message: DIYnyk 0.1.1
Parts:
- removed U$1: ILI9341, teploblinEkran:ILI9341
- added U$3: ILI9341, thermo:ILI9341
- R1, R2, R3, R4, R5, R6: value 50K -> 100K
Connections:
- net +5V renamed 5V
- net N$15 renamed SCL
- removed net N$10: R4.1, U$1.SD_MISO, U$2.IO13
- removed net N$11: U$1.T_CS, U$2.IO27
- removed net N$12: R5.1, U$1.SD_MOSI, U$2.IO26
- removed net N$13: R6.1, U$1.SD_CS, U$2.IO15
- removed net N$14: U$1.T_IRQ, U$2.SVP
- removed net N$16: C1.1, C2.1, R7.2, R8.2, U1.VDD
- removed net N$17: R7.1, U$2.IO21, U1.SDA
- removed net N$18: U$1.SD_SCK, U$2.IO14
- removed net N$7: R1.1, U$1.SDI<MOSI>, U$1.T_DIN, U$2.IO23
- removed net N$8: R2.1, U$1.SDO<MISO>, U$1.T_DO, U$2.IO19
- removed net N$9: U$1.GND, U$2.GND@38
- new net 33V: C1.1, C2.1, R7.1, R8.2, U$2.3V3, U$3.VCC, U1.VDD
- new net CLK: U$2.IO18, U$3.TFT_SCK, U$3.T_CKL
- new net CS: R3.2, U$2.IO5
- new net DC: U$2.IO16, U$3.TFT_DC
- new net LED: U$2.IO17, U$3.TFT_LED
- new net MISO: R2.2, U$2.IO19, U$3.T_DO
- new net RESET: U$2.EN, U$3.TFT_RESET
- new net SD-SCK: U$2.IO14, U$3.SD_SCK, U$3.SD_SCK_3
- new net SDA: R7.2, U$2.IO21, U1.SDA
- new net SD_CS: R6.2, U$2.IO15
- new net SD_MISO: R5.1, U$2.IO26
- new net SD_MOSI: R4.2, U$2.IO13
- new net T_CS: U$2.IO27, U$3.T_CS
- new net T_IRQ: U$2.SVN, U$3.T_IRQ
- new net V_MOSI: R1.1, U$2.IO23, U$3.T_DIN
- net GND: now also U$2.GND@38, U$3.GND; no longer U$2.GND@32
- net N$1: now also R5.2, U$3.SD_MISO, U$3.SD_MISO_3; no longer U$1.TFT_SCK, U$1.T_CKL, U$2.IO18
- net N$2: now also R4.1, U$3.SD_MOSI, U$3.SD_MOSI_3; no longer R1.2, R2.2, R3.2, R4.2, R5.2, R6.2, U$1.VCC, U$2.3V3
- net N$3: now also R6.1, U$3.SD_CS, U$3.SD_CS_3; no longer U$1.TFT_LED, U$2.IO17
- net N$4: now also R2.1, U$3.SDO<MISO>; no longer R3.1, U$1.TFT_CS, U$2.IO5
- net N$5: now also R3.1, U$3.TFT_CS; no longer U$1.TFT_RESET, U$2.EN
- net N$6: now also R1.2, U$3.SDI<MOSI>; no longer U$1.TFT_DC, U$2.IO16
Other:
- moved on the sheet: C1, C2, JP1, R1, R2, R3, R4, R5, R6, R7, R8
