File: eagle/lib/thermo.sch (EAGLE design)
At the start: 14 parts, among them U1 MLX90640ESF-BAB-000-TU

Commit message: Updated scheme 0.0.2
Parts:
- removed C1: 10U, capacitor-wima:C2,5-3
- removed C2: 100n, capacitor-wima:C2,5-3
- removed R7, R8: 1K, rcl:R-EU_0204/7
- removed U1: MLX90640ESF-BAB-000-TU, teploblinEkran:MLX90640ESF-BAB-000-TU
- added C3: 10U, capacitor-wima:C2,5-3
- added C4: 100n, capacitor-wima:C2,5-3
- added R10, R9: 1K, rcl:R-EU_0204/7
- added U2: MLX90640ESF-BAB-000-TU, teploblinEkran:MLX90640ESF-BAB-000-TU
Connections:
- net 3V3: now also C3.1, C4.1, R10.1, R9.1, U2.VDD; no longer C1.1, C2.1, R7.1, R8.1, U1.VDD
- net GND: now also C3.2, C4.2, U2.GND; no longer C1.2, C2.2, U1.GND
- net SCL: now also R9.2, U2.SCL; no longer R7.2, U1.SCL
- net SDA: now also R10.2, U2.SDA; no longer R8.2, U1.SDA
- net SD_CS: now also U$1.SD_CS_28
- net SD_MISO: now also U$1.SD_MISO_28
- net SD_MOSI: now also U$1.SD_MOSI_28
- net SD_SCK: now also U$1.SD_SCK_28

Commit message: Fixed scheme 0.1.2
Other:
- moved on the sheet: C3, C4, R10, R9, U2

Commit message: comleted
Parts:
- removed R10, R9: 1K, rcl:R-EU_0204/7
- removed U$1: ILI9341_DISPLAY_SD_MODULE, thermo:ILI9341_DISPLAY_SD_MODULE
- added R7, R8: 1K, rcl:R-EU_0204/7
- added U$3: ILI9341_DISPLAY_SD_MODULE, thermo:ILI9341_DISPLAY_SD_MODULE
Connections:
- net 3V3: now also R7.1, R8.1, U$3.VCC; no longer R10.1, R9.1, U$1.VCC
- net GND: now also U$3.GND; no longer U$1.GND
- net SCL: now also R8.2; no longer R9.2
- net SDA: now also R7.2; no longer R10.2
- net SD_CS: now also U$3.SD_CS_24, U$3.SD_CS_28, U$3.SD_CS_32; no longer U$1.SD_CS_24, U$1.SD_CS_28, U$1.SD_CS_32
- net SD_MISO: now also U$3.SD_MISO_24, U$3.SD_MISO_28, U$3.SD_MISO_32; no longer U$1.SD_MISO_24, U$1.SD_MISO_28, U$1.SD_MISO_32
- net SD_MOSI: now also U$3.SD_MOSI_24, U$3.SD_MOSI_28, U$3.SD_MOSI_32; no longer U$1.SD_MOSI_24, U$1.SD_MOSI_28, U$1.SD_MOSI_32
- net SD_SCK: now also U$3.SD_SCK_24, U$3.SD_SCK_28, U$3.SD_SCK_32; no longer U$1.SD_SCK_24, U$1.SD_SCK_28, U$1.SD_SCK_32
- net TFT_CS: now also U$3.TFT_CS; no longer U$1.TFT_CS
- net TFT_DC: now also U$3.TFT_DC; no longer U$1.TFT_DC
- net TFT_LED: now also U$3.TFT_LED; no longer U$1.TFT_LED
- net TFT_MISO: now also U$3.TFT_SDO(MISO), U$3.TOUCH_SDO(MISO); no longer U$1.TFT_SDO(MISO), U$1.TOUCH_SDO(MISO)
- net TFT_MOSI: now also U$3.TFT_SDI(MOSI), U$3.TOUCH_SDI(MOSI); no longer U$1.TFT_SDI(MOSI), U$1.TOUCH_SDI(MOSI)
- net TFT_RESET: now also U$3.TFT_RESET; no longer U$1.TFT_RESET
- net TFT_SCK: now also U$3.TFT_SCK, U$3.TOUCH_CKL(SCK); no longer U$1.TFT_SCK, U$1.TOUCH_CKL(SCK)
- net TOUCH_CS: now also U$3.TOUCH_CS; no longer U$1.TOUCH_CS
- net TOUCH_IRQ: now also U$3.TOUCH_IRQ; no longer U$1.TOUCH_IRQ
Other:
- moved on the sheet: C3, C4, JP1, R1, R2, R3, R4, R5, R6, U2
